Commit message: changed varun model

File: debug_layer/varun_description/urdf/varun.urdf (robot description, URDF)
Before this commit: robot Part1, 1 links, 0 joints
Links:
- removed link Part1
- added link varun, mass 10; collision mesh filename=package://varun_description/meshes/varun.dae; visual mesh filename=package://varun_description/meshes/varun.dae
